File: vca.kicad_sch (KiCad schematic)
At the start: 55 parts, among them U1 lm13700, U2 tl072, U3 tl072, U4 tl072, U5 tl072

Commit message: adjusted resistor values to standardize and reduce types
Parts:
- R11, R27: value 50k -> 51k
Changed lines of the file:
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@@
     (in_bom yes) (on_board yes) (fields_autoplaced)
     (property "Reference" "R27" (id 0) (at 97.79 154.3008 90))
-    (property "Value" "50k" (id 1) (at 97.79 156.5995 90))
+    (property "Value" "51k" (id 1) (at 97.79 156.5995 90))
     (property "Footprint" "" (id 2) (at 97.79 160.528 90)
       (effects (font (size 1.27 1.27)) hide)
@@
     (in_bom yes) (on_board yes) (fields_autoplaced)
     (property "Reference" "R11" (id 0) (at 99.06 46.3508 90))
-    (property "Value" "50k" (id 1) (at 99.06 48.6495 90))
+    (property "Value" "51k" (id 1) (at 99.06 48.6495 90))
     (property "Footprint" "" (id 2) (at 99.06 52.578 90)
       (effects (font (size 1.27 1.27)) hide)
